Commit message: Scene Update: Shifted all objects in scene.xml so the floor sits exactly at z=0.0
fix(scene): resolve planning failures by correcting link collision geometry.

Collision Fix: Modified collision geometry for link0 and link1 of the Panda arm.

Root Cause: The original collision meshes for the base links extended below the arm's physical base. This caused the robot to start in a collision state with the table, preventing the planner from finding any valid paths.

File: franka_description/robots/common/panda_arm.xacro (robot description, xacro)
@@ -17,5 +17,5 @@
         </geometry>
       </visual>
-      <collision>
+      <!-- <collision>
         <origin xyz="-0.075 0 0.06" rpy="0 ${pi/2} 0"/>
         <geometry>
@@ -34,4 +34,11 @@
           <sphere radius="${0.06+safety_distance}" />
         </geometry>
+      </collision> -->
+      <collision>
+        <origin xyz="-0.075 0 ${0.06 + safety_distance/2}" rpy="0 0 0"/>
+        <geometry>
+          <!-- height is base_height + safety_distance (top only, not bottom) -->
+          <box size="${0.15 + 2*safety_distance} ${0.12 + 2*safety_distance} ${0.12 + safety_distance}" />
+        </geometry>
       </collision>
     </link>
@@ -48,10 +55,10 @@
         </geometry>
       </collision>
-      <collision>
+      <!-- <collision>
         <origin xyz="0 0 -0.333" rpy="0 0 0"/>
         <geometry>
           <sphere radius="${0.06+safety_distance}" />
         </geometry>
-      </collision>
+      </collision> -->
       <collision>
         <origin xyz="0 0 -0.05" rpy="0 0 0"/>
